Commit message: Add inertial to urdf

File: pan_tilt_description/urdf/pan_tilt.urdf.xacro (robot description, xacro)
@@ -19,4 +19,9 @@
         </material>
       </visual>
+      <inertial>
+        <origin xyz="0 0 0" rpy="0 0 0"/>
+        <mass value="1"/>
+        <inertia ixx="0.01"  ixy="0"  ixz="0" iyy="0.01" iyz="0" izz="0.01" />
+      </inertial>
     </link>
     <link name="${prefix}_yaw_link">
@@ -30,4 +35,9 @@
         </material>
       </visual>
+      <inertial>
+        <origin xyz="0 0 0" rpy="0 0 0"/>
+        <mass value="1"/>
+        <inertia ixx="0.01"  ixy="0"  ixz="0" iyy="0.01" iyz="0" izz="0.01" />
+      </inertial>
     </link>
     <joint name="${prefix}_yaw_joint" type="continuous">
@@ -48,4 +58,9 @@
         </material>
       </visual>
+      <inertial>
+        <origin xyz="0 0 0" rpy="0 0 0"/>
+        <mass value="1"/>
+        <inertia ixx="0.01"  ixy="0"  ixz="0" iyy="0.01" iyz="0" izz="0.01" />
+      </inertial>
     </link>
     <joint name="${prefix}_pitch_joint" type="continuous">
@@ -56,5 +71,11 @@
       <limit lower="-1.04" upper="1.04" effort="0.0" velocity="0.0"/>
     </joint>
-    <link name="${prefix}_kinect_surface"/>
+    <link name="${prefix}_kinect_surface">
+      <inertial>
+        <origin xyz="0 0 0" rpy="0 0 0"/>
+        <mass value="1"/>
+        <inertia ixx="0.01"  ixy="0"  ixz="0" iyy="0.01" iyz="0" izz="0.01" />
+      </inertial>
+    </link>
     <joint name="${prefix}_kinect_surface_joint" type="fixed">
       <origin xyz="0.0010 0.0077 -0.022" rpy="0 0 0" />
